File: hardware/hall_effect.kicad_pcb (KiCad board)
At the start: 2 copper layers, 15 x 25 mm, 15 parts, among them P1 CON-SENSOR, U1 M24C64, U2 AH180N-W, U3 DRILL, U4 DRILL, U5 DRILL, U6 DRILL

Commit message: Add 3d information; fix EdgeCuts
Parts:
- C1, C2: footprint 0603 -> kicad-libraries:C0603
- Fiducial_Mark (x2): footprint Fiducial_Mark -> kicad-libraries:Fiducial_Mark
- G***: footprint Logo_31x31 -> kicad-libraries:Logo_31x31
- P1: footprint CON-SENSOR -> kicad-libraries:CON-SENSOR
- R1: footprint 0603 -> kicad-libraries:R0603
- U1: footprint SOIC8 -> kicad-libraries:SOIC8
- U2: footprint SC59 -> kicad-libraries:SC59
- U3, U4, U5, U6: footprint DRILL_NP -> kicad-libraries:DRILL_NP
- VAL: footprint WEEE_7mm -> kicad-libraries:WEEE_7mm
- VAL: footprint CE_5mm -> kicad-libraries:CE_5mm
Connections:
- P1 pad 1: (no net) -> Net-(P1-Pad1)
- P1 pad 10: (no net) -> Net-(P1-Pad10)
- P1 pad 8: (no net) -> Net-(P1-Pad8)
- P1 pad 9: (no net) -> Net-(P1-Pad9)
- U1 pad 7: (no net) -> Net-(U1-Pad7)
Other:
- outline, holes or cut-outs redrawn
